Commit message: Depth cloud fixed via urdf tf origins, rviz fixed without depth image topic

File: conveyor_belt/urdf/camera.urdf (robot description, URDF)
Before this commit: robot camera_robot, 15 links, 14 joints
Joints:
- joint base_leg1: origin (none) -> xyz=-0.15 0 1 rpy=0 0.1489 0
- joint base_leg2: origin (none) -> xyz=0.075 0.1299 1 rpy=0 0.1489 -2.094
- joint base_leg3: origin (none) -> xyz=0.075 -0.1299 1 rpy=0 0.1489 2.094
- joint camera_color_joint: origin (none) -> xyz=0 0 0 rpy=0 0 0
- joint camera_color_optical_joint: origin (none) -> xyz=0 0 0  rpy=-1.57 0 -1.57
- joint camera_depth_joint: origin (none) -> xyz=0 0 0 rpy=0 0 0
- joint camera_depth_optical_joint: origin (none) -> xyz=0 0 0  rpy=-1.57 0 -1.57
- joint camera_joint: origin (none) -> xyz=0 0 2.05 rpy=0 0.524 0
- joint camera_left_ir_joint: origin (none) -> xyz=0 0 0  rpy=0 0 0 
- joint camera_left_ir_optical_joint: origin (none) -> xyz=0 0 0  rpy=-1.57 0 -1.57
- joint camera_link_joint: origin (none) -> xyz=0 0.0175 0.0125  rpy=0 0 0
- joint camera_right_ir_joint: origin (none) -> xyz=0 -0.050 0  rpy=0 0 0
- joint camera_right_ir_optical_joint: origin (none) -> xyz=0 0 0  rpy=-1.57 0 -1.57
- joint top_base: origin (none) -> xyz=0 0 -2.0 rpy=0 0 0
