Commit message: Fixed belt issues

File: conveyor_belt/urdf/box.urdf (robot description, URDF)
Before this commit: robot simple_box, 1 links, 0 joints
Links:
- link box_link: mass 1.0 -> 0.1

File: conveyor_belt/urdf/cylinder.urdf (robot description, URDF)
Before this commit: robot cylinder, 1 links, 0 joints
Links:
- link link: mass 1.0 -> 0.1

File: conveyor_belt/urdf/sphere.urdf (robot description, URDF)
Before this commit: robot sphere, 1 links, 0 joints
Links:
- link link: mass 1.0 -> 0.1

Commit message: Updated belt to 10m and included side moving sections

File: conveyor_belt/urdf/box.urdf (robot description, URDF)
Before this commit: robot simple_box, 1 links, 0 joints
Links:
- link box_link: mass 0.1 -> 0.05

File: conveyor_belt/urdf/cylinder.urdf (robot description, URDF)
Before this commit: robot cylinder, 1 links, 0 joints
Links:
- link link: mass 0.1 -> 0.05

File: conveyor_belt/urdf/sphere.urdf (robot description, URDF)
Before this commit: robot sphere, 1 links, 0 joints
Links:
- link link: mass 0.1 -> 0.05

Commit message: Larger belt objects

File: conveyor_belt/urdf/box.urdf (robot description, URDF)
Before this commit: robot simple_box, 1 links, 0 joints
Links:
- link box_link: geometry collision box size=0.3 0.3 0.3; visual box size=0.3 0.3 0.3

File: conveyor_belt/urdf/cylinder.urdf (robot description, URDF)
Before this commit: robot cylinder, 1 links, 0 joints
Links:
- link link: geometry collision cylinder length=0.2 radius=0.15; visual cylinder length=0.2 radius=0.15

File: conveyor_belt/urdf/sphere.urdf (robot description, URDF)
Before this commit: robot sphere, 1 links, 0 joints
Links:
- link link: geometry collision sphere radius=0.15; visual sphere radius=0.15
